File: XTBus.sch (KiCad schematic (older format))
At the start: 29 parts, among them IC1 74LS157, IC12 74LS139, IC13 74LS245, IC14 D7201C, IC15 D8253C-5, IC2 74LS09, IC3 SN75176AP, IC4 SN75176AP, IC5 74LS123, IC6 74LS393, IC7 74LS14, IC8 74LS04, IC9 74LS11, J1 DB9_Female, J2 Bus_ISA_8bit

Commit message: modification du bus ISA. ajout de nom sur les pads
Connections:
- net labels added: ADDR_00, ADDR_01, ADDR_02, ADDR_03, ADDR_04, ADDR_05, ADDR_06, ADDR_07, IC5_8, IRQ3, RESET, vers~CS, ~IOR, ~IOW
- net labels removed: +12V, DRQ2, IC13_10, IC13_20, IC3_4, ISA_19, ISA_2, ISA_28, ISA_30, ISA_32, ISA_33, ISA_34, ISA_35, ISA_36, ISA_37, ISA_38, ISA_39, ISA_7, SMEMW, ~DACK0
- wire segments 261 -> 262
Other:
- note added: "Selecteur IRQ2,5"
- note added: "Selecteur IRQ3,6"
- note added: "selecteur IO/DRQ1,3"
- note added: "selecteur IRQ4,7"
- note added: "vers selecteur IC11\n14,12,7,10\n\n"
- note added: "vers selecteur IC11\n9,11,13,15"
- note removed: "Reset"
- moved on the sheet: C15, C16, C6, IC1, IC12A, IC12B, IC13, IC14, IC15, IC6A, IC6B, IC7E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

Commit message: les jumpers
Connections:
- net labels added: IRQ2,5, IRQ3,6, IRQ4,7
- net labels removed: IRQ3
- wire segments 262 -> 272
- no-connect marks 0 -> 16
Other:
- note added: "selecteurs IRQ"
- note removed: "Selecteur IRQ3,6"
- note removed: "selecteur IRQ4,7"
Changed lines of the file:
@@
 Comment4 ""
 $EndDescr
-Text GLabel 2750 3400 0    50   Input ~ 0
+Text GLabel 2750 4150 0    50   Input ~ 0
 ~DACK1
-Text GLabel 2750 3200 0    50   Input ~ 0
+Text GLabel 2750 3950 0    50   Input ~ 0
 ~DACK3
 $Comp
@@
 	1    0    0    -1
 $EndComp
-Wire Wire Line
-	2500 2200 2500 1750
 $Comp
 L nano:D7201C IC?
@@
 	10650 2100 10650 1300
 Wire Wire Line
-	10100 800  10100 1900
-Wire Wire Line
 	8150 1100 8100 1100
 Wire Wire Line
@@
 	1000 3150 2000 3150
 Wire Wire Line
-	2000 1900 2600 1900
+	2000 1900 2400 1900
 Connection ~ 2000 1900
-Wire Wire Line
-	2600 2500 2300 2500
 Wire Wire Line
 	900  1200 900  1300
@@
 Wire Wire Line
 	2000 1750 2000 1900
-Wire Wire Line
-	2500 1750 2000 1750
-Wire Wire Line
-	2300 2200 2500 2200
 Wire Wire Line
 	1600 1300 2000 1300
@@
 	-1   0    0    1
 $EndComp
-Wire Wire Line
-	2600 1900 2600 2500
 Text GLabel 9150 3100 2    50   Input ~ 0
 IC14_27
@@
 Wire Wire Line
 	10600 3850 10600 4600
-Wire Wire Line
-	7150 2900 7100 2900
 $Comp
 L 74xx:74LS393 IC6
@@
 Text GLabel 7450 2500 1    50   Input ~ 0
 ~IOR
-Text GLabel 2650 2800 0    50   Input ~ 0
+Text GLabel 3000 2900 0    50   Input ~ 0
 ~IOR
-Text GLabel 2650 2650 0    50   Input ~ 0
+Text GLabel 3000 2750 0    50   Input ~ 0
 ~IOW
 Wire Wire Line
-	3000 3400 2750 3400
-Wire Wire Line
-	3000 3100 2900 3100
-Wire Wire Line
-	2900 3100 2900 2800
-Wire Wire Line
-	2900 2800 2650 2800
-Wire Wire Line
-	3000 3000 2950 3000
-Wire Wire Line
-	2950 3000 2950 2650
-Wire Wire Line
-	2950 2650 2650 2650
+	3000 4150 2750 4150
 Entry Bus Bus
 	5800 2550 5900 2650
@@
 Wire Wire Line
 	6650 4350 8350 4350
-Wire Wire Line
-	7150 4600 7150 2900
 Wire Wire Line
 	6650 3900 6650 4350
@@
 	10800 800  10800 2600
 Wire Wire Line
-	2800 4700 2800 5300
-Wire Wire Line
-	1900 4700 2800 4700
-Wire Wire Line
-	4500 2700 4500 5300
-Wire Wire Line
-	2800 5300 4500 5300
-Wire Wire Line
-	4550 2800 4550 3850
+	1900 4700 1950 4700
 Text GLabel 4600 4800 2    50   Input ~ 0
 ADDR_00
@@
 	6000 3500 6000 3400
 Wire Wire Line
-	7350 3500 7350 5250
-Wire Wire Line
-	7350 5250 7600 5250
-Wire Wire Line
 	7100 3500 7350 3500
-Text GLabel 7600 5250 2    50   Input ~ 0
-IRQ3
-Text GLabel 3000 4200 0    50   Input ~ 0
-IRQ3
-Text Notes 7400 5200 0    50   ~ 0
-Selecteur IRQ3,6
 Wire Wire Line
 	7200 3400 7200 3600
-Text Notes 8050 4900 2    50   ~ 0
-selecteur IRQ4,7
 Text Notes 8900 700  0    50   ~ 0
 Selecteur IRQ2,5
@@
 	4400 3400 4600 3400
 Wire Wire Line
-	4400 2800 4550 2800
-Wire Wire Line
-	4400 2700 4500 2700
-Wire Wire Line
 	6850 1300 6850 650
 Connection ~ 6850 1300
 Wire Wire Line
 	3000 650  6850 650
-$Comp
-L nano:Bus_ISA_8bit J?
-U 1 1 61287212
-P 3700 3300
-AR Path="/61287212" Ref="J?"  Part="1"
-AR Path="/6126F7E9/61287212" Ref="J2"  Part="1"
-F 0 "J2" H 3300 1500 50  0000 C CNN
-F 1 "Bus_ISA_8bit" H 3100 1600 50  0000 C CNN
-F 2 "nano:BUS_AT_8bits" H 3700 3300 50  0001 C CNN
-F 3 "https://en.wikipedia.org/wiki/Industry_Standard_Architecture" H 3700 3300 50  0001 C CNN
-	1    3700 3300
-	1    0    0    -1
-$EndComp
-Wire Wire Line
-	3000 650  3000 2000
 Wire Wire Line
 	9600 1250 9600 600
@@
 	9600 600  2950 600
 Wire Wire Line
-	3000 2100 2950 2100
-Wire Wire Line
-	2950 600  2950 2100
+	2950 600  2950 1700
 Text GLabel 7000 1300 2    50   Input ~ 0
 C7
@@
 	6850 4700 10900 4700
 Wire Wire Line
-	10600 4600 7150 4600
+	10600 4600 7450 4600
 Wire Wire Line
 	7150 2700 7650 2700
@@
 Connection ~ 5300 3150
 Connection ~ 6650 4350
-Wire Wire Line
-	7100 4950 7900 4950
-Wire Wire Line
-	7100 3700 7100 4950
 Text GLabel 1100 4350 1    50   Input ~ 0
 IC14_32
@@
 selecteur IO/DRQ1,3
 Wire Wire Line
-	2750 3200 3000 3200
+	2750 3950 3000 3950
 Wire Wire Line
 	6000 1350 6000 1000
@@
 Wire Wire Line
 	3550 5200 2850 5200
-Wire Wire Line
-	2850 5200 2850 4500
-Wire Wire Line
-	2000 4500 2000 3150
-Wire Wire Line
-	2000 4500 2850 4500
 $Comp
 L power:GND #PWR?
@@
 Wire Wire Line
 	8450 1550 8450 1100
-Text GLabel 10100 800  0    50   Input ~ 0
-IC5_8
 Text Notes 11200 1550 1    50   ~ 0
 vers selecteur IC11\n9,11,13,15
@@
 Text Label 8600 4600 0    50   ~ 0
 vers~CS
+NoConn ~ 4300 3500
+NoConn ~ 4300 3600
+NoConn ~ 4300 3700
+NoConn ~ 4300 3800
+Wire Wire Line
+	2800 2100 2800 2250
+Text Label 2700 2000 1    50   ~ 0
+IRQ3,6
+Connection ~ 2800 2250
+Wire Wire Line
+	2800 2250 2800 2400
+Text Label 2800 2000 1    50   ~ 0
+IRQ4,7
+Text Label 2600 2200 3    50   ~ 0
+IRQ2,5
+Wire Wire Line
+	2800 2100 2900 2100
+Wire Wire Line
+	2750 2000 2900 2000
+Wire Wire Line
+	2350 1750 2350 2200
+Wire Wire Line
+	2300 2200 2350 2200
+Wire Wire Line
+	2350 1750 2000 1750
+Wire Wire Line
+	2400 2500 2400 1900
+Wire Wire Line
+	2400 2500 2300 2500
+Wire Wire Line
+	3000 1900 2950 1900
+NoConn ~ 3000 2000
+Wire Wire Line
+	2750 2000 2750 2300
+Wire Wire Line
+	2700 2000 2700 2250
+Wire Wire Line
+	2700 2250 2800 2250
+NoConn ~ 2900 2000
+NoConn ~ 3000 2300
+NoConn ~ 2900 2300
+Wire Wire Line
+	2750 2300 2900 2300
+NoConn ~ 2900 2100
+NoConn ~ 3000 2100
+NoConn ~ 3000 2200
+NoConn ~ 2900 2200
+Wire Wire Line
+	2900 2200 2600 2200
+Wire Wire Line
+	2600 2200 2600 1700
+Wire Wire Line
+	2000 3150 2850 3150
+Wire Wire Line
+	2850 3150 2850 5200
+NoConn ~ 3000 4050
+NoConn ~ 3000 4250
+NoConn ~ 2900 4250
+NoConn ~ 2900 4050
+Wire Wire Line
+	2900 4250 2400 4250
+Wire Wire Line
+	2400 4250 2400 4050
+Wire Wire Line
+	2400 4050 2900 4050
+Wire Wire Line
+	3000 4350 2400 4350
+Wire Wire Line
+	2400 4350 2400 4250
+Connection ~ 2400 4250
+Wire Wire Line
+	1950 4700 1950 4250
+Wire Wire Line
+	1950 4250 2400 4250
+Wire Wire Line
+	4400 3200 4550 3200
+Wire Wire Line
+	4550 3200 4550 3850
+Wire Wire Line
+	3000 650  3000 1800
+Wire Wire Line
+	2950 1700 2600 1700
+Connection ~ 2950 1700
+Wire Wire Line
+	2950 1700 2950 1900
+Text Label 7350 3800 3    50   ~ 0
+IRQ3,6
+Text Label 7200 3800 3    50   ~ 0
+IRQ4,7
+Wire Wire Line
+	7450 2900 7450 4600
+Wire Wire Line
+	7100 2900 7450 2900
+Wire Wire Line
+	7100 3700 7200 3700
+Wire Wire Line
+	7200 3700 7200 3800
+Wire Wire Line
+	7350 3500 7350 3800
+$Comp
+L nano:Bus_ISA_8bit J?
+U 1 1 61287212
+P 3700 3300
+AR Path="/61287212" Ref="J?"  Part="1"
+AR Path="/6126F7E9/61287212" Ref="J2"  Part="1"
+F 0 "J2" H 3300 1500 50  0000 C CNN
+F 1 "Bus_ISA_8bit" H 3100 1600 50  0000 C CNN
+F 2 "nano:BUS_AT_8bits" H 3700 3300 50  0001 C CNN
+F 3 "https://en.wikipedia.org/wiki/Industry_Standard_Architecture" H 3700 3300 50  0001 C CNN
+	1    3700 3300
+	1    0    0    -1
+$EndComp
+Wire Wire Line
+	2800 2400 3000 2400
+Text Notes 6850 4150 0    50   ~ 0
+selecteurs IRQ
+$Comp
+L power:GND #PWR?
+U 1 1 61E9BC59
+P 9950 1000
+F 0 "#PWR?" H 9950 750 50  0001 C CNN
+F 1 "GND" H 9955 827 50  0000 C CNN
+F 2 "" H 9950 1000 50  0001 C CNN
+F 3 "" H 9950 1000 50  0001 C CNN
+	1    9950 1000
+	1    0    0    -1
+$EndComp
+Wire Wire Line
+	9950 1000 9950 950
+Wire Wire Line
+	9950 950  10100 950
+Wire Wire Line
+	10100 950  10100 1900
 Wire Bus Line
 	4700 1750 4700 2450
@@
 Wire Bus Line
 	7550 3000 7550 4250
+Text Label 10100 950  0    50   ~ 0
+IC5_8
 $EndSCHEMATC
